File: 6502-computer.sch (KiCad schematic (older format))
At the start: 24 parts, among them J1 USB, P1 BUS 1, P2 BUS 2, P3 BUS 3, P5 ICP SEL, SW1 RESET, U1 WD65C02, U2 AT28C256, U3 CY7C199, U4 74HC132, U5 MXO45HS, U6 7805

Commit message: ass ginle step and improved ICP
Parts:
- removed P5: ICP SEL, symbol CONN_3X2
- added P4: ICP, symbol CONN_2
- added P5: SS, symbol CONN_2
- added R6, R7, R8: 3.3K, ~, symbol R
Connections:
- net labels added: RDY, SYNC
- wire segments 219 -> 228
- no-connect marks 7 -> 6
Other:
- note added: "FOR ICP, PULL ~RST~ L, A14 H\n1=~WE~, 2=~OE~, ~A15~=~CS"
- note added: "SEE ICP\nHEADER"
- note added: "SINGLE STEPPING\nUSUALLY LEFT NC"
- note removed: "FOR ICP, SHORT 3&5, 4&6,\nPULL ~RST~ LOW, R/~W~=~WE~, A14=~OE~"
- note removed: "FOR STD BEHAVIOUR,\nSHORT 1&3, 2&4"
- moved on the sheet: J1, U6
